File: robot_hw/mobrob_old/mobrob.kicad_pcb (KiCad board)
At the start: 2 copper layers, 35 parts, among them J1 POWER, J2 RMOTOR_OUT, J3 MCU_ROW1, J4 RMOTOR_OUT, J5 MCU_ROW2, J6 LHALL, J7 RHALL, J8 IMU, J9 UT, U1 L293D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

Commit message: Massive dump
Parts:
- removed D9: D_Schottky, Package_TO_SOT_SMD:TO-252-2_TabPin1
- J4: value RMOTOR_OUT -> LMOTOR_OUT
- R1, R6: value R -> 33k
- R2, R5: value R -> 15k
- R3, R4: value R -> 150
- moved D4 115.8 mm to (230.5, 116.0), turned to 90 degrees
- moved J9 110.4 mm to (171.0, 117.0), turned to 180 degrees
- moved D6 108.7 mm to (205.1, 83.0), turned to 90 degrees
- moved J3 102.7 mm to (138.2, 104.0)
- moved J5 102.1 mm to (138.2, 84.6)
- moved J4 94.3 mm to (217.8, 115.0), turned to 180 degrees
- moved D8 90.0 mm to (225.4, 105.9), turned to 270 degrees
- moved D7 89.1 mm to (205.1, 105.9), turned to 270 degrees
- moved D3 87.3 mm to (200.0, 116.0), turned to 90 degrees
- moved D1 87.1 mm to (230.5, 72.8), turned to 270 degrees
- moved D2 86.6 mm to (200.0, 72.8), turned to 270 degrees
- moved D5 82.3 mm to (225.4, 83.0), turned to 90 degrees
- moved J1 80.1 mm to (180.1, 73.0), turned to 0 degrees
- moved C4 76.7 mm to (229.0, 93.0), turned to 270 degrees
- moved C3 71.1 mm to (201.0, 96.0), turned to 90 degrees
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Connections:
- C1 pad 1: Net-(C1-Pad1) -> +12V
- C3 pad 2: Net-(C3-Pad2) -> +12V
- U1 pad 1: EN1,2 -> 1,2EN
- U1 pad 8: Net-(C3-Pad2) -> +12V
- U1 pad 9: EN3,4 -> 3,4EN
- U2 pad 1: Net-(C1-Pad1) -> +12V
Routing:
- net +5V: track 0.00 -> 65.8 mm
- net +12V: track 0.00 -> 44.8 mm
- net Net-(D1-Pad2): track 0.00 -> 41.7 mm
- net Net-(D3-Pad2): track 0.00 -> 31.8 mm
- net Net-(D4-Pad2): track 0.00 -> 31.5 mm
- net LED_STATUS: track 0.00 -> 21.8 mm
- net Net-(D2-Pad2): track 0.00 -> 11.2 mm
- net Net-(J6-Pad2): track 0.00 -> 10.6 mm
- net Net-(D11-Pad1): track 0.00 -> 3.47 mm
- net (no net): vias 0 -> 12
Other:
- board outline added: 100 x 54 mm
- net class Default: via_drill 0.4 -> 0.5
- rule trace_min: 0.2 -> 0.25
